File: Schematic/LED_Dimmer/LED_Dimmer.kicad_sch (KiCad schematic)
At the start: 26 parts, among them J1 From PSU, J2 LED Spots, J3 To microsocope, J4 LED Ring, U1 AL8861Y-13, U2 AL8861Y-13

Commit message: Adjusted mounting hole position
Parts:
- R1: value 200mΩ 0.5W -> 200mΩ 0.25W
- R3: value 200mΩ 0.5W -> 120mΩ 0.25W
- R4: value 10kΩ -> 9.1kΩ
Changed lines of the file:
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@@
       (effects (font (size 1.27 1.27)))
     )
-    (property "Value" "200mΩ 0.5W" (at 118.745 36.195 90)
+    (property "Value" "200mΩ 0.25W" (at 118.745 36.195 90)
       (effects (font (size 1.27 1.27)))
     )
@@
       (effects (font (size 1.27 1.27)))
     )
-    (property "Value" "200mΩ 0.5W" (at 118.745 88.9 90)
+    (property "Value" "120mΩ 0.25W" (at 118.745 88.9 90)
       (effects (font (size 1.27 1.27)))
     )
@@
       (effects (font (size 1.27 1.27)))
     )
-    (property "Value" "10kΩ" (at 93.98 96.52 90)
-      (effects (font (size 1.27 1.27)))
-    )
+    (property "Value" "9.1kΩ" (at 93.98 96.52 90)
+      (effects (font (size 1.27 1.27)))
+    )

Commit message: New PCB layout
Parts:
- added C5: 22µF, Resistor_SMD:R_0805_2012Metric_Pad1.20x1.40mm_HandSolder, symbol Device:C
- J1: renamed from J2; footprint myDevices:KF2510-2P -> myDevices:KF2510-2P-Angle
- J2: renamed from J1; footprint myDevices:KF2510-2P -> myDevices:KF2510-2P-Angle
- J3: renamed from J4; footprint myDevices:KF2510-2P -> myDevices:KF2510-2P-Angle
- J4: renamed from J3; footprint myDevices:KF2510-2P -> myDevices:KF2510-2P-Angle
- R4: value 9.1kΩ -> 10kΩ
- renumbered C5 to C6, C6 to C7
Connections:
- net +5V: now also C5.1
- net GND: now also C5.2
Other:
- moved on the sheet: H1, H2, H3, H4
